Commit message: feat(visual): geometria por primitivas dimensionadas desde la tabla D-H
Cilindros y esferas cuyo largo sale de a_i o d_i, no de mallas externas.
link_5 sin cilindro: a_5 = d_5 = 0, firma de la muneca esferica.
El cuerpo se declara antes de la articulacion porque RViz aplica a todo
el link el primer material que encuentra.
Cadena verificada tras anadir geometria: 3.68e-16 m.

File: urdf/irb120.urdf (robot description, URDF)
Before this commit: robot irb120, 8 links, 7 joints
Links:
- link base_link: geometry visual cylinder length=0.04 radius=0.11
- link link_1: geometry collision cylinder length=0.290000 radius=0.0570; visual cylinder length=0.290000 radius=0.0600
- link link_2: geometry collision cylinder length=0.270000 radius=0.0522; visual cylinder length=0.270000 radius=0.0550
- link link_3: geometry collision cylinder length=0.070000 radius=0.0427; visual cylinder length=0.070000 radius=0.0450
- link link_4: geometry collision cylinder length=0.302000 radius=0.0361; visual cylinder length=0.302000 radius=0.0380
- link link_5: geometry visual sphere radius=0.0368
- link link_6: geometry collision cylinder length=0.072000 radius=0.0266; visual cylinder length=0.072000 radius=0.0280
- link tool0: geometry visual cylinder length=0.012 radius=0.031
